File: MiniDrone_aDat.kicad_sch (KiCad schematic)
At the start: 8 parts

Commit message: 5/7/2025
Parts:
- removed Mt1, Mt2, Mt3, Mt4: ~, Motor_Screws:720DCMotor, symbol Motor_ScrewsHole:720DCMotor
- removed Scr1, Scr2, Scr3, Scr4: ~, Motor_Screws:ScrewM2, symbol Motor_ScrewsHole:ScrewM2
Other:
- note removed: "MechanicPart"

Commit message: 4/7/2025
Parts:
- added Mt1, Mt2, Mt3, Mt4: ~, Motor_Screws:720DCMotor, symbol Motor_ScrewsHole:720DCMotor
- added Scr1, Scr2, Scr3, Scr4: ~, Motor_Screws:PillarScrew5mmM3, symbol Motor_ScrewsHole:PillarScrews5mmM3
Connections:
- new net GND: Mt1.GND, Mt2.GND, Mt3.GND, Mt4.GND, Scr1.GND, Scr2.GND, Scr3.GND, Scr4.GND
Other:
- note added: "MechanicPart"

Commit message: 4/7/2025
Parts:
- removed Scr1, Scr2, Scr3, Scr4: ~, Motor_Screws:PillarScrew5mmM3, symbol Motor_ScrewsHole:PillarScrews5mmM3
- added Scr1, Scr2, Scr3, Scr4: ~, Motor_Screws:ScrewM2, symbol Motor_ScrewsHole:ScrewM2
