File: MiniDrone_aDat.kicad_pcb (KiCad board)
At the start: 2 copper layers, 50 parts, among them J1 Screw_Terminal_01x02, J10 Conn_01x04, J2 Screw_Terminal_01x02, J3 Screw_Terminal_01x02, J4 Screw_Terminal_01x02, J5 Screw_Terminal_01x02, J6 Conn_01x08, J7 Conn_01x04, J8 Conn_02x04_Counter_Clockwise, J9 Conn_01x04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

Commit message: 2/7/2025
Parts:
- C13, C15, C3, J1, J2, J3, J4, U3, U5: moved to B.Cu
- D1: footprint Capacitor_SMD:C_0201_0603Metric -> Capacitor_SMD:C_0603_1608Metric
- J10: footprint Connector_PinHeader_1.00mm:PinHeader_1x04_P1.00mm_Vertical -> Connector_PinHeader_2.54mm:PinHeader_1x04_P2.54mm_Vertical; moved to B.Cu
- J5: footprint TerminalBlock:TerminalBlock_MaiXu_MX126-5.0-02P_1x02_P5.00mm -> TerminalBlock:TerminalBlock_Xinya_XY308-2.54-2P_1x02_P2.54mm_Horizontal
- J6: footprint Connector_PinHeader_1.00mm:PinHeader_1x08_P1.00mm_Vertical -> Connector_PinHeader_2.54mm:PinHeader_1x08_P2.54mm_Vertical; moved to B.Cu
- J7, J9: footprint Connector_PinHeader_1.00mm:PinHeader_1x04_P1.00mm_Vertical -> Connector_PinHeader_2.54mm:PinHeader_1x04_P2.54mm_Vertical
- J8: footprint Connector_PinHeader_1.00mm:PinHeader_2x04_P1.00mm_Vertical -> Connector_PinHeader_2.54mm:PinHeader_2x04_P2.54mm_Vertical; moved to B.Cu
- moved J4 65.6 mm to (77.0, 125.5), turned to 135 degrees
- moved C21 64.1 mm to (72.5, 128.0), turned to -45 degrees
- moved J3 61.1 mm to (124.5, 122.5), turned to -135 degrees
- moved U3 50.6 mm to (100.0, 116.0), turned to -90 degrees
- moved J7 49.5 mm to (117.3, 117.6), turned to 180 degrees
- moved D2 47.7 mm to (102.9, 116.2), turned to -90 degrees
- moved C23 45.2 mm to (127.0, 127.0), turned to 45 degrees
- moved C19 44.2 mm to (72.0, 72.0), turned to -135 degrees
- moved J5 41.7 mm to (118.7, 101.5), turned to 90 degrees
- moved J1 41.3 mm to (124.5, 74.0), turned to -45 degrees
- moved C1 35.9 mm to (116.5, 104.6)
- moved C15 35.8 mm to (109.0, 116.7), turned to -90 degrees
- moved U5 31.2 mm to (100.0, 85.0), turned to 90 degrees
- moved C8 31.1 mm to (116.5, 106.6)
- moved R7 30.6 mm to (106.4, 114.9)
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Routing:
- net +3V3: track 0.00 -> 190.4 mm, vias 0 -> 5
- net /TopLevelDesign/PB12: track 0.00 -> 78.5 mm
- net /TopLevelDesign/PB14: track 0.00 -> 77.5 mm
- net /TopLevelDesign/PB15: track 0.00 -> 62.3 mm
- net Vin: track 0.00 -> 54.4 mm, vias 0 -> 1
- net /TopLevelDesign/PA12: track 0.00 -> 52.1 mm
- net /TopLevelDesign/PB13: track 0.00 -> 47.1 mm, vias 0 -> 1
- net /TopLevelDesign/HBridge/H2_OUTB1: track 0.00 -> 40.7 mm
- net /TopLevelDesign/HBridge/H1_OUTB1: track 0.00 -> 39.8 mm
- net /TopLevelDesign/SWDIO: track 0.00 -> 39.7 mm
- net /TopLevelDesign/PA15: track 0.00 -> 39.3 mm
- net /TopLevelDesign/HBridge/H1_OUTA2: track 0.00 -> 39.1 mm
- net /TopLevelDesign/HBridge/H2_OUTA2: track 0.00 -> 38.9 mm
- net /TopLevelDesign/HBridge/H1_OUTA1: track 0.00 -> 29.8 mm
- net /TopLevelDesign/MCU/PA0: track 0.00 -> 29.7 mm, vias 0 -> 2
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- added copper zone on B.Cu, net GND
- added copper zone on F.Cu, net GND
Other:
- board outline added: 100 x 100 mm

Commit message: 4/7/2025
Parts:
- added Mt1: ~, Motor_Screws:720DCMotor, F.Cu at (137.8, 62.4)
- added Mt2: ~, Motor_Screws:720DCMotor, F.Cu at (62.9, 62.8)
- added Mt3: ~, Motor_Screws:720DCMotor, F.Cu at (62.9, 137.8)
- added Mt4: ~, Motor_Screws:720DCMotor, F.Cu at (137.9, 137.8)
- added Scr1: ~, Motor_Screws:PillarScrew5mmM3, B.Cu at (132.0, 68.7)
- added Scr2: ~, Motor_Screws:PillarScrew5mmM3, B.Cu at (68.7, 68.7)
- added Scr3: ~, Motor_Screws:PillarScrew5mmM3, B.Cu at (132.0, 132.0)
- added Scr4: ~, Motor_Screws:PillarScrew5mmM3, B.Cu at (68.7, 131.9)
- moved C13 0.66 mm to (109.0, 83.3)
- moved R5 0.38 mm to (110.3, 103.6)
- moved J10 0.23 mm to (120.3, 87.2)
Routing:
- net Vin: track 54.4 -> 99.8 mm, vias 1 -> 2
- net +3V3: track 190.4 -> 219.3 mm
- net /TopLevelDesign/HBridge/H1_INA1: track 14.8 -> 17.0 mm
- net /TopLevelDesign/HBridge/H1_OUTB1: track 39.8 -> 41.7 mm
- net /TopLevelDesign/MCU/PA0: track 29.7 -> 31.3 mm
- net /TopLevelDesign/PB10: track 25.4 -> 23.8 mm
- net /TopLevelDesign/HBridge/H1_INB1: track 15.3 -> 16.6 mm
- net /TopLevelDesign/SWDIO: track 39.7 -> 40.9 mm
- net /TopLevelDesign/HBridge/H2_OUTB1: track 40.7 -> 39.6 mm
- net /TopLevelDesign/PA12: track 52.1 -> 53.0 mm
- net /TopLevelDesign/PB15: track 62.3 -> 63.1 mm
- net /TopLevelDesign/PB14: track 77.5 -> 78.2 mm
- net /TopLevelDesign/HBridge/H1_OUTA1: track 29.8 -> 29.1 mm
- net /TopLevelDesign/PB4: track 16.4 -> 15.8 mm
- net /TopLevelDesign/PB11: track 19.2 -> 18.6 mm
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Other:
- outline, holes or cut-outs redrawn

Commit message: 4/7/2025
Parts:
- moved R9 0.45 mm to (110.9, 91.6)
- moved J8 0.29 mm to (85.8, 96.2)
Connections:
- J8 pad 2: /TopLevelDesign/PA12 -> +3V3
- J8 pad 3: /TopLevelDesign/PB13 -> /TopLevelDesign/PA12
- J8 pad 4: /TopLevelDesign/PB14 -> /TopLevelDesign/PB12
- J8 pad 5: /TopLevelDesign/PA15 -> /TopLevelDesign/PB13
- J8 pad 7: /TopLevelDesign/PB12 -> /TopLevelDesign/PB14
- J8 pad 8: +3V3 -> /TopLevelDesign/PA15
Routing:
- net /TopLevelDesign/PB13: track 46.7 -> 81.9 mm, vias 1 -> 0
- net /TopLevelDesign/PB12: track 78.6 -> 93.8 mm
- net /TopLevelDesign/SWCLK: track 29.5 -> 40.5 mm
- net /TopLevelDesign/PA15: track 39.3 -> 49.7 mm, vias 0 -> 1
- net +3V3: track 219.3 -> 210.8 mm
- net /TopLevelDesign/PA12: track 53.0 -> 59.6 mm
- net /TopLevelDesign/PB14: track 78.2 -> 73.0 mm
- net Net-(U4-+): track 11.1 -> 10.1 mm
- net /TopLevelDesign/HBridge/H1_INB2: track 18.7 -> 18.1 mm
- net GND: vias 36 -> 47

Commit message: 4/7/2025
Parts:
- Scr1, Scr2, Scr3, Scr4: footprint Motor_Screws:PillarScrew5mmM3 -> Motor_Screws:ScrewM2
- moved J10 7.64 mm to (119.5, 94.8), turned to 0 degrees
- moved J3 2.68 mm to (126.3, 124.5)
- moved C23 2.68 mm to (128.8, 129.0)
Connections:
- Scr1 pad GND: GND -> (no net)
- Scr2 pad GND: GND -> (no net)
- Scr3 pad GND: GND -> (no net)
- Scr4 pad GND: GND -> (no net)
Routing:
- net /TopLevelDesign/HBridge/H2_OUTB2: track 25.8 -> 38.6 mm
- net /TopLevelDesign/HBridge/H2_OUTA2: track 38.5 -> 33.9 mm
- net /TopLevelDesign/PB11: track 18.6 -> 22.9 mm
- net /TopLevelDesign/PB10: track 23.8 -> 22.0 mm

Commit message: 5/7/2025
Parts:
- added Scr10: ~, Motor_Screws:ScrewM2, F.Cu at (143.9, 143.1)
- added Scr11: ~, Motor_Screws:ScrewM2, F.Cu at (62.9, 70.8)
- added Scr12: ~, Motor_Screws:ScrewM2, F.Cu at (56.9, 143.3)
- added Scr13: ~, Motor_Screws:ScrewM2, F.Cu at (137.9, 129.8)
- added Scr14: ~, Motor_Screws:ScrewM2, F.Cu at (143.0, 56.6)
- added Scr15: ~, Motor_Screws:ScrewM2, F.Cu at (62.9, 129.8)
- added Scr16: ~, Motor_Screws:ScrewM2, F.Cu at (129.9, 137.8)
- added Scr5: ~, Motor_Screws:ScrewM2, F.Cu at (57.5, 56.8)
- added Scr6: ~, Motor_Screws:ScrewM2, F.Cu at (137.9, 70.8)
- added Scr7: ~, Motor_Screws:ScrewM2, F.Cu at (70.9, 137.8)
- added Scr8: ~, Motor_Screws:ScrewM2, F.Cu at (70.9, 62.8)
- added Scr9: ~, Motor_Screws:ScrewM2, F.Cu at (129.8, 62.8)
- moved Scr4 11.9 mm to (77.1, 123.5)
- moved Scr2 11.7 mm to (77.0, 76.9)
- moved Scr3 11.5 mm to (124.3, 123.5)
- moved Scr1 11.4 mm to (124.1, 76.9)
- moved C21 5.30 mm to (68.8, 131.8)
- moved J4 5.30 mm to (73.3, 129.3)
- moved C19 4.60 mm to (68.8, 68.7)
- moved J2 4.60 mm to (71.3, 73.2)
- moved C23 4.42 mm to (132.0, 132.0)
- moved J3 4.42 mm to (129.5, 127.5)
- moved J1 4.17 mm to (127.6, 71.2)
- moved C17 4.17 mm to (132.1, 68.7)
Connections:
- Scr1 pad GND: (no net) -> GND
- Scr2 pad GND: (no net) -> GND
- Scr3 pad GND: (no net) -> GND
- Scr4 pad GND: (no net) -> GND
Routing:
- net /TopLevelDesign/HBridge/H2_OUTA1: track 26.7 -> 41.5 mm
- net /TopLevelDesign/HBridge/H1_OUTA1: track 29.1 -> 43.4 mm
- net /TopLevelDesign/HBridge/H1_OUTB2: track 27.6 -> 41.1 mm
- net /TopLevelDesign/HBridge/H2_OUTA2: track 33.9 -> 39.4 mm
- net /TopLevelDesign/HBridge/H2_OUTB2: track 38.6 -> 42.0 mm
- net /TopLevelDesign/PB12: track 93.8 -> 91.5 mm
- net /TopLevelDesign/HBridge/H1_OUTB1: track 41.7 -> 39.4 mm
- net /TopLevelDesign/PB13: track 81.9 -> 79.8 mm
- net +3V3: track 210.5 -> 209.1 mm
- net /TopLevelDesign/HBridge/H2_OUTB1: track 39.6 -> 38.2 mm
- net /TopLevelDesign/HBridge/H1_OUTA2: track 39.1 -> 38.2 mm
- net /TopLevelDesign/PB14: track 73.0 -> 72.2 mm
- net /TopLevelDesign/PB15: track 63.6 -> 62.9 mm
- net GND: vias 47 -> 51

Commit message: 6/7/2025
Parts:
- moved Scr13 2.97 mm to (140.2, 127.9)
- moved C17 2.97 mm to (134.3, 66.8)
- moved C2 2.97 mm to (105.4, 90.1)
- moved C23 2.97 mm to (134.3, 130.1)
- moved J3 2.97 mm to (131.8, 125.6)
- moved Mt1 2.97 mm to (140.0, 60.5)
- moved Scr10 2.97 mm to (146.2, 141.2)
- moved Scr16 2.97 mm to (132.1, 135.9)
- moved Scr4 2.97 mm to (79.4, 121.6)
- moved Scr6 2.97 mm to (140.2, 69.0)
- moved Scr9 2.97 mm to (132.1, 60.9)
- moved J4 2.97 mm to (75.6, 127.5)
- moved C1 2.97 mm to (118.8, 102.7)
- moved C10 2.97 mm to (87.8, 115.2)
- moved C11 2.97 mm to (115.3, 97.2)
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Other:
- outline, holes or cut-outs redrawn
- board text added: "3V3"
- board text added: "Au:Crypt"
- board text added: "CE"
- board text added: "CK"
- board text added: "CSN"
- board text added: "DroneADat"
- board text added: "GND"
- board text added: "IQR"
- board text added: "MISO"
- board text added: "MOSI"
- board text added: "RX"
- board text added: "SCK"
- board text added: "SWCLK"
- board text added: "SWDIO"
- board text added: "TX"
