File: TopLevelDesign.kicad_sch (KiCad schematic)
At the start: 10 parts, among them J1 Screw_Terminal_01x02, J10 Conn_01x04, J2 Screw_Terminal_01x02, J3 Screw_Terminal_01x02, J4 Screw_Terminal_01x02, J5 Screw_Terminal_01x02, J6 Conn_01x08, J7 Conn_01x04, J8 Conn_02x04_Counter_Clockwise, J9 Conn_01x04

Commit message: 2/7/2025
Parts:
- J10, J7, J9: footprint Connector_PinHeader_1.00mm:PinHeader_1x04_P1.00mm_Vertical -> Connector_PinHeader_2.54mm:PinHeader_1x04_P2.54mm_Vertical
- J5: footprint TerminalBlock:TerminalBlock_MaiXu_MX126-5.0-02P_1x02_P5.00mm -> TerminalBlock:TerminalBlock_Xinya_XY308-2.54-2P_1x02_P2.54mm_Horizontal
- J6: footprint Connector_PinHeader_1.00mm:PinHeader_1x08_P1.00mm_Vertical -> Connector_PinHeader_2.54mm:PinHeader_1x08_P2.54mm_Vertical
- J8: footprint Connector_PinHeader_1.00mm:PinHeader_2x04_P1.00mm_Vertical -> Connector_PinHeader_2.54mm:PinHeader_2x04_P2.54mm_Vertical

Commit message: 4/7/2025
Connections:
- net +3V3: now also J8.2 (Pin_2); no longer J8.8 (Pin_8)
- net PA12: now also J8.3 (Pin_3); no longer J8.2 (Pin_2)
- net PA15: now also J8.8 (Pin_8); no longer J8.5 (Pin_5)
- net PB12: now also J8.4 (Pin_4); no longer J8.7 (Pin_7)
- net PB13: now also J8.5 (Pin_5); no longer J8.3 (Pin_3)
- net PB14: now also J8.7 (Pin_7); no longer J8.4 (Pin_4)

Commit message: 5/7/2025
Parts:
- added Mt1, Mt2, Mt3, Mt4: ~, Motor_Screws:720DCMotor, symbol Motor_ScrewsHole:720DCMotor
- added Scr1, Scr10, Scr11, Scr12, Scr13, Scr14, Scr15, Scr16, Scr2, Scr3, Scr4, Scr5, Scr6, Scr7, Scr8, Scr9: ~, Motor_Screws:ScrewM2, symbol Motor_ScrewsHole:ScrewM2
Connections:
- net GND: now also Mt1.GND, Mt2.GND, Mt3.GND, Mt4.GND, Scr1.GND, Scr10.GND, Scr11.GND, Scr12.GND, Scr13.GND, Scr14.GND, Scr15.GND, Scr16.GND, Scr2.GND, Scr3.GND, Scr4.GND, Scr5.GND, Scr6.GND, Scr7.GND, Scr8.GND, Scr9.GND
Other:
- note added: "MechanicPart"

Commit message: 6/7/2025
Changed lines of the file:
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@@
 	(wire
 		(pts
-			(xy 69.85 29.21) (xy 69.85 27.94)
-		)
-		(stroke
-			(width 0)
-			(type default)
-		)
-	)
-	(wire
-		(pts
 			(xy 87.63 151.13) (xy 92.71 151.13)
 		)
@@
 	)
 	(label "PA15"
-		(at 69.85 27.94 180)
+		(at 69.85 29.21 180)
 		(effects
 			(font
